Commit message: feat(rover_description): gate sim_mode/drive_model in URDF; fix steering joints + Select artifact
Co-Authored-By: Claude Opus 4.7 <noreply@anthropic.com>

File: ros2_ws/src/rover_description/urdf/robot.urdf.xacro (robot description, xacro)
@@ -3,9 +3,21 @@
     <xacro:arg name="use_ros2_control" default="true" />
     <xacro:arg name="sim_mode" default="false" />
+    <xacro:arg name="drive_model" default="diff" />   <!-- diff | ackermann -->
     <xacro:include filename="robot_core.xacro" />
-    <xacro:include filename="ros2_control.xacro" />
-    <xacro:include filename="lidar.xacro" />
-    <xacro:include filename="imu.xacro" />
-    <xacro:include filename="camera.xacro" />
-    <!-- <xacro:include filename="depth_camera.xacro" /> -->
+    <xacro:if value="$(arg sim_mode)">
+        <xacro:include filename="gz_sensors.xacro" />
+        <xacro:include filename="gz_joint_state.xacro" />
+        <xacro:if value="${'$(arg drive_model)' == 'ackermann'}">
+            <xacro:include filename="gz_ackermann.xacro" />
+        </xacro:if>
+        <xacro:unless value="${'$(arg drive_model)' == 'ackermann'}">
+            <xacro:include filename="gz_diff_drive.xacro" />
+        </xacro:unless>
+    </xacro:if>
+    <xacro:unless value="$(arg sim_mode)">
+        <xacro:include filename="ros2_control.xacro" />
+        <xacro:include filename="lidar.xacro" />
+        <xacro:include filename="imu.xacro" />
+        <xacro:include filename="camera.xacro" />
+    </xacro:unless>
 </robot>

File: ros2_ws/src/rover_description/urdf/robot_core.xacro (robot description, xacro)
@@ -43,5 +43,5 @@
     <link
         name="base_link" />
-    <!-- BASE_FOOTPRINT LINK -->Select <joint name="base_footprint_joint" type="fixed">
+    <!-- BASE_FOOTPRINT LINK --><joint name="base_footprint_joint" type="fixed">
         <parent link="base_link" />
         <child link="base_footprint" />
@@ -145,5 +145,5 @@
         <axis xyz="0 0 1" />
         <dynamics damping="0.2" />
-        <limit lower="-0.454" upper="0.384" effort="100.0" velocity="0.0" />
+        <limit lower="-0.454" upper="0.384" effort="100.0" velocity="2.0" />
     </joint>
     <link
@@ -174,5 +174,5 @@
         <axis xyz="0 0 1" />
         <dynamics damping="0.2" />
-        <limit lower="-0.384" upper="0.454" effort="100.0" velocity="0.0" />
+        <limit lower="-0.384" upper="0.454" effort="100.0" velocity="2.0" />
     </joint>
     <link
