Commit message: fix(rover_description): define sensor frames in gz_sensors.xacro
Sim mode excludes the real lidar/imu/camera.xacro (Classic plugins), which also defined the laser_frame/imu_link/camera_link links. Without them the gz sensors attached to nothing and published no data. Define the frames here (poses matching the real ones) so sim is self-contained. Verified: /scan 9.9Hz, /imu 49Hz, /camera 18.8Hz headless.

Co-Authored-By: Claude Opus 4.7 <noreply@anthropic.com>

File: ros2_ws/src/rover_description/urdf/gz_sensors.xacro (robot description, xacro)
@@ -1,4 +1,35 @@
 <?xml version="1.0"?>
 <robot xmlns:xacro="http://www.ros.org/wiki/xacro">
+  <!-- Sensor frames. In sim_mode the real lidar/imu/camera.xacro are NOT included
+       (they carry Gazebo Classic plugins), so the sensor links are defined here so
+       sim is self-contained. Poses match the real lidar/imu/camera.xacro frames. -->
+  <joint name="laser_joint" type="fixed">
+    <parent link="chassis"/><child link="laser_frame"/>
+    <origin xyz="0.175 0.0 0.153" rpy="0 0 0"/>
+  </joint>
+  <link name="laser_frame">
+    <visual><geometry><cylinder radius="0.05" length="0.04"/></geometry>
+      <material name="red"><color rgba="1 0 0 1"/></material></visual>
+    <inertial><mass value="0.1"/>
+      <inertia ixx="1e-4" ixy="0" ixz="0" iyy="1e-4" iyz="0" izz="1e-4"/></inertial>
+  </link>
+  <joint name="imu_joint" type="fixed">
+    <parent link="chassis"/><child link="imu_link"/>
+    <origin xyz="0.208 0.03 0.0" rpy="0 0 0"/>
+  </joint>
+  <link name="imu_link">
+    <visual><geometry><box size="0.02 0.02 0.01"/></geometry></visual>
+    <inertial><mass value="0.01"/>
+      <inertia ixx="1e-6" ixy="0" ixz="0" iyy="1e-6" iyz="0" izz="1e-6"/></inertial>
+  </link>
+  <joint name="camera_joint" type="fixed">
+    <parent link="chassis"/><child link="camera_link"/>
+    <origin xyz="0.24 0.0 0.13" rpy="0 0 0"/>
+  </joint>
+  <link name="camera_link">
+    <visual><geometry><box size="0.01 0.03 0.03"/></geometry></visual>
+    <inertial><mass value="0.01"/>
+      <inertia ixx="1e-6" ixy="0" ixz="0" iyy="1e-6" iyz="0" izz="1e-6"/></inertial>
+  </link>
   <!-- 2D LiDAR -> /scan -->
   <gazebo reference="laser_frame">
